Commit message: format code1

File: simlate_gazebo/simulate_robot/urdf/robot_with_realsense.urdf.xacro (robot description, xacro)
@@ -5,11 +5,11 @@
 	<link name="camera0_link">
         <visual>
-          <origin xyz=" 0 0 0 " rpy="0 0 0" />
-          <geometry>
-          <sphere radius="0.01" />
-          </geometry>
-          <material name="black">
-          <color rgba="0 0 0 0.95"/>
-          </material>
+            <origin xyz=" 0 0 0 " rpy="0 0 0" />
+            <geometry>
+                <sphere radius="0.01" />
+            </geometry>
+            <material name="black">
+                <color rgba="0 0 0 0.95"/>
+            </material>
         </visual>
     </link>
@@ -29,349 +29,356 @@
         </material>
       </visual>
-      </link>
-      <joint name="camera1_joint" type="fixed">
-        <origin xyz="0.00 0 0.5" rpy="0 0 1.0471975511965976"/>
+    </link>
+    <joint name="camera1_joint" type="fixed">
+        <origin xyz="0.0 0 0.5" rpy="0 0 1.0471975511965976"/>
         <parent link="base_link"/>
         <child link="camera1_link"/>
       </joint>
-      <link name="camera2_link">
-        <visual>
-          <origin xyz=" 0 0 0 " rpy="0 0 0" />
-          <geometry>
-          <sphere radius="0.01" />
-          </geometry>
-          <material name="black">
-          <color rgba="0 0 0 0.95"/>
-          </material>
-        </visual>
-        </link>
-        <joint name="camera2_joint" type="fixed">
-          <origin xyz="0.00 0 0.5" rpy="0 0 2.0943951023931953"/>
-          <parent link="base_link"/>
-          <child link="camera2_link"/>
-        </joint>
-        <link name="camera3_link">
-          <visual>
-            <origin xyz=" 0 0 0 " rpy="0 0 0" />
-            <geometry>
-            <sphere radius="0.01" />
-            </geometry>
-            <material name="black">
-            <color rgba="0 0 0 0.95"/>
-            </material>
-          </visual>
-          </link>
-          <joint name="camera3_joint" type="fixed">
-            <origin xyz="0.00 0 0.5" rpy="0 0 3.141592653589793"/>
-            <parent link="base_link"/>
-            <child link="camera3_link"/>
-          </joint>
-          <link name="camera4_link">
-            <visual>
-              <origin xyz=" 0 0 0 " rpy="0 0 0" />
-              <geometry>
-              <sphere radius="0.01" />
-              </geometry>
-              <material name="black">
-              <color rgba="0 0 0 0.95"/>
-              </material>
-            </visual>
-            </link>
-            <joint name="camera4_joint" type="fixed">
-              <origin xyz="0.00 0 0.5" rpy="0 0 -2.0943951023931953"/>
-              <parent link="base_link"/>
-              <child link="camera4_link"/>
-            </joint>
-            <link name="camera5_link">
-              <visual>
-                <origin xyz=" 0 0 0 " rpy="0 0 0" />
-                <geometry>
-                <sphere radius="0.01" />
-                </geometry>
-                <material name="black">
-                <color rgba="0 0 0 0.95"/>
-                </material>
-              </visual>
-              </link>
-              <joint name="camera5_joint" type="fixed">
-                <origin xyz="0.00 0 0.5" rpy="0 0 -1.0471975511965976 "/>
-                <parent link="base_link"/>
-                <child link="camera5_link"/>
-              </joint>
-        <gazebo reference="camera0_link">
+    <link name="camera2_link">
+        <visual>
+            <origin xyz=" 0 0 0 " rpy="0 0 0" />
+            <geometry>
+                <sphere radius="0.01" />
+            </geometry>
+            <material name="black">
+                <color rgba="0 0 0 0.95"/>
+            </material>
+        </visual>
+    </link>
+    <joint name="camera2_joint" type="fixed">
+        <origin xyz="0.0 0 0.5" rpy="0 0 2.0943951023931953"/>
+        <parent link="base_link"/>
+        <child link="camera2_link"/>
+    </joint>
+    <link name="camera3_link">
+        <visual>
+            <origin xyz=" 0 0 0 " rpy="0 0 0" />
+            <geometry>
+                <sphere radius="0.01" />
+            </geometry>
+            <material name="black">
+                <color rgba="0 0 0 0.95"/>
+            </material>
+        </visual>
+    </link>
+    <joint name="camera3_joint" type="fixed">
+        <origin xyz="0.0 0 0.5" rpy="0 0 3.141592653589793"/>
+        <parent link="base_link"/>
+        <child link="camera3_link"/>
+    </joint>
+    <link name="camera4_link">
+        <visual>
+            <origin xyz=" 0 0 0 " rpy="0 0 0" />
+            <geometry>
+                <sphere radius="0.01" />
+            </geometry>
+            <material name="black">
+                <color rgba="0 0 0 0.95"/>
+            </material>
+        </visual>
+    </link>
+    <joint name="camera4_joint" type="fixed">
+        <origin xyz="0.0 0 0.5" rpy="0 0 -2.0943951023931953"/>
+        <parent link="base_link"/>
+        <child link="camera4_link"/>
+    </joint>
+    <link name="camera5_link">
+        <visual>
+            <origin xyz=" 0 0 0 " rpy="0 0 0" />
+            <geometry>
+                <sphere radius="0.01" />
+            </geometry>
+            <material name="black">
+                <color rgba="0 0 0 0.95"/>
+            </material>
+        </visual>
+    </link>
+    <joint name="camera5_joint" type="fixed">
+        <origin xyz="0.0 0 0.5" rpy="0 0 -1.0471975511965976 "/>
+        <parent link="base_link"/>
+        <child link="camera5_link"/>
+    </joint>
+    <!-- camera simulator plug-in -->
+    <gazebo reference="camera0_link">  <!--加载相机的插件, 下面配置相机参数-->
 		<turnGravityOff>false</turnGravityOff>
 		<sensor type="depth" name="realsense_depth">
-		<update_rate>30.0</update_rate>
-		<camera>
-		<!-- 75x65 degree FOV for the depth sensor -->
-		<horizontal_fov>1.5184351666666667</horizontal_fov>
-		<vertical_fov>1.0122901111111111</vertical_fov>
-		<image>
-		<width>640</width>
-		<height>480</height>
-		<!-- TODO: check what format the Realsense hardware delivers and set this to match! -->
-		<format>RGB8</format>
-		</image>
-		<clip>
-		<!-- give the color sensor a maximum range of 50m so that the simulation renders nicely -->
-		<near>0.01</near>
-		<far>50.0</far>
-		</clip>
-		</camera>
-		<plugin name="kinect_controller" filename="libgazebo_ros_openni_kinect.so">
-		<baseline>0.2</baseline>
-		<alwaysOn>true</alwaysOn>
-		<updateRate>30</updateRate>
-		<cameraName>camera0</cameraName>
-		<imageTopicName>color/image_raw</imageTopicName>
-		<cameraInfoTopicName>color/camera_info</cameraInfoTopicName>
-		<depthImageTopicName>depth/image_rect_raw</depthImageTopicName>
-		<depthImageInfoTopicName>depth/camera_info</depthImageInfoTopicName>
-		<pointCloudTopicName>depth/color/points</pointCloudTopicName>
-		<frameName>camera0_link</frameName>
-		<pointCloudCutoff>0.1</pointCloudCutoff>
-		<pointCloudCutoffMax>10.0</pointCloudCutoffMax>
-		<distortionK1>0.00000001</distortionK1>
-		<distortionK2>0.00000001</distortionK2>
-		<distortionK3>0.00000001</distortionK3>
-		<distortionT1>0.00000001</distortionT1>
-		<distortionT2>0.00000001</distortionT2>
-		<CxPrime>0</CxPrime>
-		<Cx>0</Cx>
-		<Cy>0</Cy>
-		<focalLength>0</focalLength>
-		<hackBaseline>0</hackBaseline>
-		</plugin>
+            <update_rate>30.0</update_rate>
+            <camera>
+                <!-- 75x65 degree FOV for the depth sensor, 相机 水平/俯仰 视场角 -->
+                <horizontal_fov>1.5184351666666667</horizontal_fov>
+                <vertical_fov>1.0122901111111111</vertical_fov>
+                <image>
+                    <width>640</width> <!--像素宽度  u-->
+                    <height>480</height> <!--像素高度 v-->
+                    <!-- TODO: check what format the Realsense hardware delivers and set this to match! -->
+                    <format>RGB8</format>
+                </image>
+                <clip>
+                    <!-- give the color sensor a maximum range of 50m so that the simulation renders nicely -->
+                    <near>0.01</near> <!--最近拍摄距离-->
+                    <far>50.0</far> <!--最远拍摄距离-->
+                </clip>
+                <!--相机噪声-->
+                <!-- <noise>
+                    <type>gaussian</type>
+                    <mean>0.0</mean>
+                    <stddev>0.000</stddev>
+                </noise> -->
+            </camera>
+            <plugin name="kinect_controller" filename="libgazebo_ros_openni_kinect.so">
+                <baseline>0.2</baseline>
+                <alwaysOn>true</alwaysOn>
+                <updateRate>30</updateRate>
+                <cameraName>camera0</cameraName>
+                <imageTopicName>color/image_raw</imageTopicName>
+                <cameraInfoTopicName>color/camera_info</cameraInfoTopicName>
+                <depthImageTopicName>depth/image_rect_raw</depthImageTopicName>
+                <depthImageInfoTopicName>depth/camera_info</depthImageInfoTopicName>
+                <pointCloudTopicName>depth/color/points</pointCloudTopicName>
+                <frameName>camera0_link</frameName>
+                <pointCloudCutoff>0.1</pointCloudCutoff>
+                <pointCloudCutoffMax>10.0</pointCloudCutoffMax>
+                <distortionK1>0.00000001</distortionK1>
+                <distortionK2>0.00000001</distortionK2>
+                <distortionK3>0.00000001</distortionK3>
+                <distortionT1>0.00000001</distortionT1>
+                <distortionT2>0.00000001</distortionT2>
+                <CxPrime>0</CxPrime>
+                <Cx>0</Cx>
+                <Cy>0</Cy>
+                <focalLength>0</focalLength>
+                <hackBaseline>0</hackBaseline>
+            </plugin>
 		</sensor>
 	</gazebo>
     <gazebo reference="camera1_link">
-			<turnGravityOff>false</turnGravityOff>
-			<sensor type="depth" name="realsense_depth">
-			<update_rate>30.0</update_rate>
-			<camera>
-			<!-- 75x65 degree FOV for the depth sensor -->
-			<horizontal_fov>1.5184351666666667</horizontal_fov>
-			<vertical_fov>1.0122901111111111</vertical_fov>
-			<image>
-			<width>640</width>
-			<height>480</height>
-			<!-- TODO: check what format the Realsense hardware delivers and set this to match! -->
-			<format>RGB8</format>
-			</image>
-			<clip>
-			<!-- give the color sensor a maximum range of 50m so that the simulation renders nicely -->
-			<near>0.01</near>
-			<far>50.0</far>
-			</clip>
-			</camera>
-			<plugin name="kinect_controller" filename="libgazebo_ros_openni_kinect.so">
-			<baseline>0.2</baseline>
-			<alwaysOn>true</alwaysOn>
-			<updateRate>30</updateRate>
-			<cameraName>camera1</cameraName>
-			<imageTopicName>color/image_raw</imageTopicName>
-			<cameraInfoTopicName>color/camera_info</cameraInfoTopicName>
-			<depthImageTopicName>depth/image_rect_raw</depthImageTopicName>
-			<depthImageInfoTopicName>depth/camera_info</depthImageInfoTopicName>
-			<pointCloudTopicName>depth/color/points</pointCloudTopicName>
-			<frameName>camera1_link</frameName>
-			<pointCloudCutoff>0.1</pointCloudCutoff>
-			<pointCloudCutoffMax>10.0</pointCloudCutoffMax>
-			<distortionK1>0.00000001</distortionK1>
-			<distortionK2>0.00000001</distortionK2>
-			<distortionK3>0.00000001</distortionK3>
-			<distortionT1>0.00000001</distortionT1>
-			<distortionT2>0.00000001</distortionT2>
-			<CxPrime>0</CxPrime>
-			<Cx>0</Cx>
-			<Cy>0</Cy>
-			<focalLength>0</focalLength>
-			<hackBaseline>0</hackBaseline>
-			</plugin>
-			</sensor>
-			</gazebo>
-            <gazebo reference="camera2_link">
-				<turnGravityOff>false</turnGravityOff>
-				<sensor type="depth" name="realsense_depth">
-				<update_rate>30.0</update_rate>
-				<camera>
-				<!-- 75x65 degree FOV for the depth sensor -->
-				<horizontal_fov>1.5184351666666667</horizontal_fov>
-				<vertical_fov>1.0122901111111111</vertical_fov>
-				<image>
-				<width>640</width>
-				<height>480</height>
-				<!-- TODO: check what format the Realsense hardware delivers and set this to match! -->
-				<format>RGB8</format>
-				</image>
-				<clip>
-				<!-- give the color sensor a maximum range of 50m so that the simulation renders nicely -->
-				<near>0.01</near>
-				<far>50.0</far>
-				</clip>
-				</camera>
-				<plugin name="kinect_controller" filename="libgazebo_ros_openni_kinect.so">
-				<baseline>0.2</baseline>
-				<alwaysOn>true</alwaysOn>
-				<updateRate>30</updateRate>
-				<cameraName>camera2</cameraName>
-				<imageTopicName>color/image_raw</imageTopicName>
-				<cameraInfoTopicName>color/camera_info</cameraInfoTopicName>
-				<depthImageTopicName>depth/image_rect_raw</depthImageTopicName>
-				<depthImageInfoTopicName>depth/camera_info</depthImageInfoTopicName>
-				<pointCloudTopicName>depth/color/points</pointCloudTopicName>
-				<frameName>camera2_link</frameName>
-				<pointCloudCutoff>0.1</pointCloudCutoff>
-				<pointCloudCutoffMax>10.0</pointCloudCutoffMax>
-				<distortionK1>0.00000001</distortionK1>
-				<distortionK2>0.00000001</distortionK2>
-				<distortionK3>0.00000001</distortionK3>
-				<distortionT1>0.00000001</distortionT1>
-				<distortionT2>0.00000001</distortionT2>
-				<CxPrime>0</CxPrime>
-				<Cx>0</Cx>
-				<Cy>0</Cy>
-				<focalLength>0</focalLength>
-				<hackBaseline>0</hackBaseline>
-				</plugin>
-				</sensor>
-				</gazebo>
-				<gazebo reference="camera3_link">
-					<turnGravityOff>false</turnGravityOff>
-					<sensor type="depth" name="realsense_depth">
-					<update_rate>30.0</update_rate>
-					<camera>
-					<!-- 75x65 degree FOV for the depth sensor -->
-					<horizontal_fov>1.5184351666666667</horizontal_fov>
-					<vertical_fov>1.0122901111111111</vertical_fov>
-					<image>
-					<width>640</width>
-					<height>480</height>
-					<!-- TODO: check what format the Realsense hardware delivers and set this to match! -->
-					<format>RGB8</format>
-					</image>
-					<clip>
-					<!-- give the color sensor a maximum range of 50m so that the simulation renders nicely -->
-					<near>0.01</near>
-					<far>50.0</far>
-					</clip>
-					</camera>
-					<plugin name="kinect_controller" filename="libgazebo_ros_openni_kinect.so">
-					<baseline>0.2</baseline>
-					<alwaysOn>true</alwaysOn>
-					<updateRate>30</updateRate>
-					<cameraName>camera3</cameraName>
-					<imageTopicName>color/image_raw</imageTopicName>
-					<cameraInfoTopicName>color/camera_info</cameraInfoTopicName>
-					<depthImageTopicName>depth/image_rect_raw</depthImageTopicName>
-					<depthImageInfoTopicName>depth/camera_info</depthImageInfoTopicName>
-					<pointCloudTopicName>depth/color/points</pointCloudTopicName>
-					<frameName>camera3_link</frameName>
-					<pointCloudCutoff>0.1</pointCloudCutoff>
-					<pointCloudCutoffMax>10.0</pointCloudCutoffMax>
-					<distortionK1>0.00000001</distortionK1>
-					<distortionK2>0.00000001</distortionK2>
-					<distortionK3>0.00000001</distortionK3>
-					<distortionT1>0.00000001</distortionT1>
-					<distortionT2>0.00000001</distortionT2>
-					<CxPrime>0</CxPrime>
-					<Cx>0</Cx>
-					<Cy>0</Cy>
-					<focalLength>0</focalLength>
-					<hackBaseline>0</hackBaseline>
-					</plugin>
-					</sensor>
-					</gazebo>
-					<gazebo reference="camera4_link">
-						<turnGravityOff>false</turnGravityOff>
-						<sensor type="depth" name="realsense_depth">
-						<update_rate>30.0</update_rate>
-						<camera>
-						<!-- 75x65 degree FOV for the depth sensor -->
-						<horizontal_fov>1.5184351666666667</horizontal_fov>
-						<vertical_fov>1.0122901111111111</vertical_fov>
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